Commit message: Replace robot description and meshes

File: outdoor_ws/src/outdoor_description/src/description/off_road_urdf.urdf (robot description, URDF)
Before this commit: robot outdoor_description, 9 links, 8 joints
Links:
- removed link FL_trail_link
- removed link FL_wheel_link
- removed link FR_trail_link
- removed link FR_wheel_link
- removed link RL_trail_link
- removed link RL_wheel_link
- removed link RR_trail_link
- removed link RR_wheel_link
- added link W1_l, mass 16.9385252789344; collision mesh filename=package://outdoor_description/src/description/meshes/W1_l.S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; visual mesh filename=package://outdoor_description/src/description/meshes/W1_l.S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
- added link W2_l, mass 16.9385252782885; collision mesh filename=package://outdoor_description/src/description/meshes/W2_l.S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; visual mesh filename=package://outdoor_description/src/description/meshes/W2_l.S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
- added link W3_l, mass 16.9385252831856; collision mesh filename=package://outdoor_description/src/description/meshes/W3_l.S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; visual mesh filename=package://outdoor_description/src/description/meshes/W3_l.S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
- added link W4_l, mass 16.9385252734549; collision mesh filename=package://outdoor_description/src/description/meshes/W4_l.S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; visual mesh filename=package://outdoor_description/src/description/meshes/W4_l.S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
- added link sm1_l, mass 0.7158068478374; collision mesh filename=package://outdoor_description/src/description/meshes/sm1_l.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; visual mesh filename=package://outdoor_description/src/description/meshes/sm1_l.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
- added link sm2_l, mass 0.715806847837399; collision mesh filename=package://outdoor_description/src/description/meshes/sm2_l.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; visual mesh filename=package://outdoor_description/src/description/meshes/sm2_l.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
- added link sm3_l, mass 0.715806847837399; collision mesh filename=package://outdoor_description/src/description/meshes/sm3_l.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; visual mesh filename=package://outdoor_description/src/description/meshes/sm3_l.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
- added link sm4_l, mass 0.715806847837399; collision mesh filename=package://outdoor_description/src/description/meshes/sm4_l.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; visual mesh filename=package://outdoor_description/src/description/meshes/sm4_l.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
- added link su1_l, mass 0.7158068478374; collision mesh filename=package://outdoor_description/src/description/meshes/su1_l.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; visual mesh filename=package://outdoor_description/src/description/meshes/su1_l.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
- added link su2_l, mass 0.715806847837399; collision mesh filename=package://outdoor_description/src/description/meshes/su2_l.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; visual mesh filename=package://outdoor_description/src/description/meshes/su2_l.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
- added link su3_l, mass 0.715806847837399; collision mesh filename=package://outdoor_description/src/description/meshes/su3_l.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; visual mesh filename=package://outdoor_description/src/description/meshes/su3_l.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
- added link su4_l, mass 0.715806847837399; collision mesh filename=package://outdoor_description/src/description/meshes/su4_l.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; visual mesh filename=package://outdoor_description/src/description/meshes/su4_l.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
- added link tu1_l, mass 10.2132979097438; collision mesh filename=package://outdoor_description/src/description/meshes/tu1_l.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; visual mesh filename=package://outdoor_description/src/description/meshes/tu1_l.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
- added link tu2_l, mass 7.72532312777463; collision mesh filename=package://outdoor_description/src/description/meshes/tu2_l.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; visual mesh filename=package://outdoor_description/src/description/meshes/tu2_l.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
- added link tu3_l, mass 10.2132979014202; collision mesh filename=package://outdoor_description/src/description/meshes/tu3_l.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; visual mesh filename=package://outdoor_description/src/description/meshes/tu3_l.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
- added link tu4_l, mass 7.72532312777463; collision mesh filename=package://outdoor_description/src/description/meshes/tu4_l.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; visual mesh filename=package://outdoor_description/src/description/meshes/tu4_l.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
- added link w1_l, mass 16.9385252789344; collision mesh filename=package://outdoor_description/src/description/meshes/W1_l.S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; visual mesh filename=package://outdoor_description/src/description/meshes/W1_l.S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
- added link w2_l, mass 16.9385252782884; collision mesh filename=package://outdoor_description/src/description/meshes/W2_l.S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; visual mesh filename=package://outdoor_description/src/description/meshes/W2_l.S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
- added link w3_l, mass 16.9385252831856; collision mesh filename=package://outdoor_description/src/description/meshes/W3_l.S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; visual mesh filename=package://outdoor_description/src/description/meshes/W3_l.S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
- added link w4_l, mass 16.9385252734549; collision mesh filename=package://outdoor_description/src/description/meshes/W4_l.S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; visual mesh filename=package://outdoor_description/src/description/meshes/W4_l.S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
- link base_link: mass 80.0 -> 81.8728040761975; geometry collision mesh filename=package://outdoor_description/src/description/meshes/base_l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; visual mesh filename=package://outdoor_description/src/description/meshes/base_l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
Joints:
- removed joint FL_trail_joint
- removed joint FL_wheel_joint
- removed joint FR_trail_joint
- removed joint FR_wheel_joint
- removed joint RL_trail_joint
- removed joint RL_wheel_joint
- removed joint RR_trail_joint
- removed joint RR_wheel_joint
- added joint W1_j: type continuous, parent tu1_l, child W1_l, origin xyz=0.26738 -0.229 -0.21986 rpy=0 0 0, axis 0 1 0
- added joint W2_j: type continuous, parent tu2_l, child W2_l, origin xyz=-0.26738 -0.229 -0.21986 rpy=0 0 0, axis 0 1 0
- added joint W3_j: type continuous, parent tu3_l, child W3_l, origin xyz=-0.26738 0.229 -0.21986 rpy=0 0 0, axis 0 1 0
- added joint W4_j: type continuous, parent tu4_l, child W4_l, origin xyz=0.26738 0.229 -0.21986 rpy=0 0 0, axis 0 1 0
- added joint sm1_j: type prismatic, parent su1_l, child sm1_l, origin xyz=-0.084601 0 -0.10067 rpy=0 0 0, axis 0.64336 0 0.76557, limit lower=-0.05 upper=0.05 effort=2000 velocity=0.5
- added joint sm2_j: type prismatic, parent su2_l, child sm2_l, origin xyz=0.084601 0 -0.10067 rpy=0 0 0, axis -0.64336 0 0.76557, limit lower=-0.05 upper=0.05 effort=2000 velocity=0.5
- added joint sm3_j: type prismatic, parent su3_l, child sm3_l, origin xyz=0.084601 0 -0.10067 rpy=0 0 0, axis -0.64336 0 0.76557, limit lower=-0.05 upper=0.05 effort=2000 velocity=0.5
- added joint sm4_j: type prismatic, parent su4_l, child sm4_l, origin xyz=-0.084601 0 -0.10067 rpy=0 0 0, axis 0.64336 0 0.76557, limit lower=-0.05 upper=0.05 effort=2000 velocity=0.5
- added joint su1_j: type continuous, parent base_link, child su1_l, origin xyz=0.805 -0.404 0.295 rpy=0 0 0, axis 0 1 0
- added joint su2_j: type continuous, parent base_link, child su2_l, origin xyz=-0.515 -0.405 0.295 rpy=0 0 0, axis 0 1 0
- added joint su3_j: type continuous, parent base_link, child su3_l, origin xyz=-0.515 0.405 0.295 rpy=0 0 0, axis 0 1 0
- added joint su4_j: type continuous, parent base_link, child su4_l, origin xyz=0.805 0.404 0.295 rpy=0 0 0, axis 0 1 0
- added joint tu1_j: type continuous, parent base_link, child tu1_l, origin xyz=0.33 -0.354 0.215 rpy=0 0 0, axis 0 1 0
- added joint tu2_j: type continuous, parent base_link, child tu2_l, origin xyz=-0.04 -0.354 0.215 rpy=0 0 0, axis 0 1 0
- added joint tu3_j: type continuous, parent base_link, child tu3_l, origin xyz=-0.04 0.354 0.215 rpy=0 0 0, axis 0 1 0
- added joint tu4_j: type continuous, parent base_link, child tu4_l, origin xyz=0.33 0.354 0.215 rpy=0 0 0, axis 0 1 0
- added joint w1_j: type continuous, parent sm1_l, child w1_l, origin xyz=-0.12302 -0.179 -0.19919 rpy=0 0 0, axis 0 1 0
- added joint w2_j: type continuous, parent sm2_l, child w2_l, origin xyz=0.12302 -0.178 -0.19919 rpy=0 0 0, axis 0 1 0
- added joint w3_j: type continuous, parent sm3_l, child w3_l, origin xyz=0.12302 0.178 -0.19919 rpy=0 0 0, axis 0 1 0
- added joint w4_j: type continuous, parent sm4_l, child w4_l, origin xyz=-0.12302 0.179 -0.19919 rpy=0 0 0, axis 0 1 0

File: outdoor_ws/src/outdoor_description/src/description/off_road_urdf.urdf.xacro (robot description, xacro)
@@ -1,3 +1,3 @@
-<?xml version="1.0"?>
+<?xml version="1.0" encoding="utf-8"?>
 <robot xmlns:xacro="http://www.ros.org/wiki/xacro" name="outdoor_description">
   <link
@@ -5,63 +5,651 @@
     <inertial>
       <origin
-        xyz="-8.17927536369341E-17 -1.3950931901084E-15 0.130545650801935"
-        rpy="0 0 0" />
-      <mass
-        value="150.8233509085438" />
-      <inertia
-        ixx="0.265440261208668"
-        ixy="-2.10459838722132E-17"
-        ixz="-1.53164849370567E-18"
-        iyy="0.496368289840211"
-        iyz="-8.4667989116219E-18"
-        izz="0.727766670019649" />
-    </inertial>
-    <visual>
-      <origin
-        xyz="0 0 0"
-        rpy="0 0 0" />
-      <geometry>
-        <mesh
-          filename="package://outdoor_description/src/description/meshes/chasis_link.STL" />
-      </geometry>
-      <material
-        name="">
-        <color
-          rgba="0.898039215686275 0.917647058823529 0.929411764705882 1" />
-      </material>
-    </visual>
-    <collision>
-      <origin
-        xyz="0 0 0"
-        rpy="0 0 0" />
-      <geometry>
-        <mesh
-          filename="package://outdoor_description/src/description/meshes/chasis_link.STL" />
-      </geometry>
-    </collision>
-  </link>
-  <link
-    name="RR_shock_link">
-    <inertial>
-      <origin
-        xyz="0.0763011366291501 -0.127044297188698 -0.0299999999999999"
+        xyz="0.146261722213942 0.000543929627490959 0.206998435056227"
+        rpy="0 0 0" />
+      <mass
+        value="81.8728040761975" />
+      <inertia
+        ixx="0.928332742280751"
+        ixy="-0.000538381152275935"
+        ixz="7.82462972412944E-05"
+        iyy="2.12205079983374"
+        iyz="3.95382316209524E-06"
+        izz="2.87255178322061" />
+    </inertial>
+    <visual>
+      <origin
+        xyz="0 0 0"
+        rpy="0 0 0" />
+      <geometry>
+        <mesh
+          filename="package://outdoor_description/src/description/meshes/base_link.STL" />
+      </geometry>
+      <material
+        name="">
+        <color
+          rgba="0.752941176470588 0.752941176470588 0.752941176470588 1" />
+      </material>
+    </visual>
+    <collision>
+      <origin
+        xyz="0 0 0"
+        rpy="0 0 0" />
+      <geometry>
+        <mesh
+          filename="package://outdoor_description/src/description/meshes/base_link.STL" />
+      </geometry>
+    </collision>
+  </link>
+  <link
+    name="tu1_l">
+    <inertial>
+      <origin
+        xyz="0.147362309153983 -0.0333159854188 -0.1211687926663"
+        rpy="0 0 0" />
+      <mass
+        value="10.2132979097438" />
+      <inertia
+        ixx="0.0358725371406297"
+        ixy="1.21406315693586E-05"
+        ixz="0.0375003251759691"
+        iyy="0.085464141095508"
+        iyz="-9.48193435836396E-06"
+        izz="0.0506422080598156" />
+    </inertial>
+    <visual>
+      <origin
+        xyz="0 0 0"
+        rpy="0 0 0" />
+      <geometry>
+        <mesh
+          filename="package://outdoor_description/src/description/meshes/tu1_l.STL" />
+      </geometry>
+      <material
+        name="">
+        <color
+          rgba="0.752941176470588 0.752941176470588 0.752941176470588 1" />
+      </material>
+    </visual>
+    <collision>
+      <origin
+        xyz="0 0 0"
+        rpy="0 0 0" />
+      <geometry>
+        <mesh
+          filename="package://outdoor_description/src/description/meshes/tu1_l.STL" />
+      </geometry>
+    </collision>
+  </link>
+  <joint
+    name="tu1_j"
+    type="continuous">
+    <origin
+      xyz="0.33 -0.354 0.215"
+      rpy="0 0 0" />
+    <parent
+      link="base_link" />
+    <child
+      link="tu1_l" />
+    <axis
+      xyz="0 1 0" />
+  </joint>
+  <link
+    name="W1_l">
+    <inertial>
+      <origin
+        xyz="1.71696358072237E-05 0.025264976547993 2.02005059561465E-06"
+        rpy="0 0 0" />
+      <mass
+        value="16.9385252789344" />
+      <inertia
+        ixx="0.513537561453538"
+        ixy="1.43363347826961E-05"
+        ixz="-6.77351136120244E-06"
+        iyy="0.891763002094289"
+        iyz="3.03339596888524E-06"
+        izz="0.513567792828017" />
+    </inertial>
+    <visual>
+      <origin
+        xyz="0 0 0"
+        rpy="0 0 0" />
+      <geometry>
+        <mesh
+          filename="package://outdoor_description/src/description/meshes/W1_l.STL" />
+      </geometry>
+      <material
+        name="">
+        <color
+          rgba="0.752941176470588 0.752941176470588 0.752941176470588 1" />
+      </material>
+    </visual>
+    <collision>
+      <origin
+        xyz="0 0 0"
+        rpy="0 0 0" />
+      <geometry>
+        <mesh
+          filename="package://outdoor_description/src/description/meshes/W1_l.STL" />
+      </geometry>
+    </collision>
+  </link>
+  <joint
+    name="W1_j"
+    type="continuous">
+    <origin
+      xyz="0.26738 -0.229 -0.21986"
+      rpy="0 0 0" />
+    <parent
+      link="tu1_l" />
+    <child
+      link="W1_l" />
+    <axis
+      xyz="0 1 0" />
+  </joint>
+  <link
+    name="tu2_l">
+    <inertial>
+      <origin
+        xyz="-0.137021532460763 -0.0195472382042864 -0.105386640443532"
+        rpy="0 0 0" />
+      <mass
+        value="7.72532312777463" />
+      <inertia
+        ixx="0.0263090204959749"
+        ixy="-1.1837838277264E-05"
+        ixz="-0.0295137315066913"
+        iyy="0.0639279889046924"
+        iyz="-9.73341041293776E-06"
+        izz="0.0385789482600205" />
+    </inertial>
+    <visual>
+      <origin
+        xyz="0 0 0"
+        rpy="0 0 0" />
+      <geometry>
+        <mesh
+          filename="package://outdoor_description/src/description/meshes/tu2_l.STL" />
+      </geometry>
+      <material
+        name="">
+        <color
+          rgba="0.752941176470588 0.752941176470588 0.752941176470588 1" />
+      </material>
+    </visual>
+    <collision>
+      <origin
+        xyz="0 0 0"
+        rpy="0 0 0" />
+      <geometry>
+        <mesh
+          filename="package://outdoor_description/src/description/meshes/tu2_l.STL" />
+      </geometry>
+    </collision>
+  </link>
+  <joint
+    name="tu2_j"
+    type="continuous">
+    <origin
+      xyz="-0.04 -0.354 0.215"
+      rpy="0 0 0" />
+    <parent
+      link="base_link" />
+    <child
+      link="tu2_l" />
+    <axis
+      xyz="0 1 0" />
+  </joint>
+  <link
+    name="W2_l">
+    <inertial>
+      <origin
+        xyz="1.57026386815029E-05 0.0252649765331265 -7.22875534110018E-06"
+        rpy="0 0 0" />
+      <mass
+        value="16.9385252782885" />
+      <inertia
+        ixx="0.513539751870816"
+        ixy="1.38143287927479E-05"
+        ixz="1.03596150509659E-05"
+        iyy="0.891763001369152"
+        iyz="-4.88646576774158E-06"
+        izz="0.51356560120949" />
+    </inertial>
+    <visual>
+      <origin
+        xyz="0 0 0"
+        rpy="0 0 0" />
+      <geometry>
+        <mesh
+          filename="package://outdoor_description/src/description/meshes/W2_l.STL" />
+      </geometry>
+      <material
+        name="">
+        <color
+          rgba="0.752941176470588 0.752941176470588 0.752941176470588 1" />
+      </material>
+    </visual>
+    <collision>
+      <origin
+        xyz="0 0 0"
+        rpy="0 0 0" />
+      <geometry>
+        <mesh
+          filename="package://outdoor_description/src/description/meshes/W2_l.STL" />
+      </geometry>
+    </collision>
+  </link>
+  <joint
+    name="W2_j"
+    type="continuous">
+    <origin
+      xyz="-0.26738 -0.229 -0.21986"
+      rpy="0 0 0" />
+    <parent
+      link="tu2_l" />
+    <child
+      link="W2_l" />
+    <axis
+      xyz="0 1 0" />
+  </joint>
+  <link
+    name="tu3_l">
+    <inertial>
+      <origin
+        xyz="-0.147362309060457 0.033315985364701 -0.121168792605429"
+        rpy="0 0 0" />
+      <mass
+        value="10.2132979014202" />
+      <inertia
+        ixx="0.035872537136603"
+        ixy="1.21406317571704E-05"
+        ixz="-0.0375003251787922"
+        iyy="0.0854641410781346"
+        iyz="9.48193521425474E-06"
+        izz="0.0506422080461984" />
+    </inertial>
+    <visual>
+      <origin
+        xyz="0 0 0"
+        rpy="0 0 0" />
+      <geometry>
+        <mesh
+          filename="package://outdoor_description/src/description/meshes/tu3_l.STL" />
+      </geometry>
+      <material
+        name="">
+        <color
+          rgba="0.752941176470588 0.752941176470588 0.752941176470588 1" />
+      </material>
+    </visual>
+    <collision>
+      <origin
+        xyz="0 0 0"
+        rpy="0 0 0" />
+      <geometry>
+        <mesh
+          filename="package://outdoor_description/src/description/meshes/tu3_l.STL" />
+      </geometry>
+    </collision>
+  </link>
+  <joint
+    name="tu3_j"
+    type="continuous">
+    <origin
+      xyz="-0.04 0.354 0.215"
+      rpy="0 0 0" />
+    <parent
+      link="base_link" />
+    <child
+      link="tu3_l" />
+    <axis
+      xyz="0 1 0" />
+  </joint>
+  <link
+    name="W3_l">
+    <inertial>
+      <origin
+        xyz="1.28236511909852E-05 -0.0252649764628815 1.15891516132491E-05"
+        rpy="0 0 0" />
+      <mass
+        value="16.9385252831856" />
+      <inertia
+        ixx="0.513547983602694"
+        ixy="-1.17227568826066E-05"
+        ixz="-1.58860807859731E-05"
+        iyy="0.891763001235492"
+        iyz="-8.79424995869041E-06"
+        izz="0.5135573693724" />
+    </inertial>
+    <visual>
+      <origin
+        xyz="0 0 0"
+        rpy="0 0 0" />
+      <geometry>
+        <mesh
+          filename="package://outdoor_description/src/description/meshes/W3_l.STL" />
+      </geometry>
+      <material
+        name="">
+        <color
+          rgba="0.752941176470588 0.752941176470588 0.752941176470588 1" />
+      </material>
+    </visual>
+    <collision>
+      <origin
+        xyz="0 0 0"
+        rpy="0 0 0" />
+      <geometry>
+        <mesh
+          filename="package://outdoor_description/src/description/meshes/W3_l.STL" />
+      </geometry>
+    </collision>
+  </link>
+  <joint
+    name="W3_j"
+    type="continuous">
+    <origin
+      xyz="-0.26738 0.229 -0.21986"
+      rpy="0 0 0" />
+    <parent
+      link="tu3_l" />
+    <child
+      link="W3_l" />
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